File: schmittpulsegenerator/schmittpulsegenerator.kicad_pcb (KiCad board)
At the start: 2 copper layers, 53 x 30 mm, 16 parts, among them J1 Conn_Coaxial, J2 Conn_01x02_Male, U1 74HC14

Commit message: datasheets
Other:
- rule pad_to_mask_clearance: 0.05 -> 0
Changed lines of the file:
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@@
-(kicad_pcb (version 20171130) (host pcbnew 5.1.2-f72e74a~84~ubuntu18.04.1)
+(kicad_pcb (version 20171130) (host pcbnew "(5.1.2)-1")
   (general
     (thickness 1.6)
@@
     (pad_size 15.24 15.24)
     (pad_drill 9.65)
-    (pad_to_mask_clearance 0.05)
-    (solder_mask_min_width 0.05)
+    (pad_to_mask_clearance 0)
     (aux_axis_origin 0 0)
     (visible_elements 7FFFFFFF)
     (pcbplotparams
-      (layerselection 0x00000_7fffffff)
+      (layerselection 0x00080_7ffffffe)
       (usegerberextensions false)
       (usegerberattributes false)
@@
       (hpglpenspeed 20)
       (hpglpendiameter 15.000000)
-      (psnegative true)
+      (psnegative false)
       (psa4output false)
       (plotreference true)
