File: voightfocuser/_autosave-voightfocuser.sch (KiCad schematic (older format))
At the start: 10 parts

Commit message: added parts
Parts:
- removed U?: DRV8848, Package_SO:TSSOP-16-1EP_4.4x5mm_P0.65mm, symbol Driver_Motor:DRV8848
- added U?: DRV8825, Package_SO:HTSSOP-28-1EP_4.4x9.7mm_P0.65mm_EP3.4x9.5mm_Mask2.4x6.17mm_ThermalVias, symbol JeffLibrary:DRV8825
Connections:
- net labels added: GNDC, GNDD, VDD, ~RESET
- net labels removed: GND, GNDA
- wire segments 26 -> 17
Other:
- note added: "Voight Focuser"
- moved on the sheet: SW?
Changed lines of the file:
@@
 U 1 1 5CDAD9A2
 P 800 2600
-F 0 "J?" H 857 3067 50  0000 C CNN
-F 1 "USB_B_Micro" H 857 2976 50  0000 C CNN
+F 0 "J?" H 650 3050 50  0000 C CNN
+F 1 "USB_B_Micro" H 850 2950 50  0000 C CNN
 F 2 "" H 950 2550 50  0001 C CNN
 F 3 "~" H 950 2550 50  0001 C CNN
@@
 	1    0    0    -1
 $EndComp
-Text GLabel 1900 1300 2    50   UnSpc ~ 0
-GNDA
-Text GLabel 1100 1150 2    50   UnSpc ~ 0
-GNDA
-Text GLabel 850  3000 2    50   UnSpc ~ 0
-GND
 Wire Wire Line
 	800  3000 850  3000
-Text GLabel 4900 6250 2    50   UnSpc ~ 0
-GND
 Wire Wire Line
 	4800 6200 4800 6250
@@
 Wire Wire Line
 	4900 3250 4950 3250
-Wire Wire Line
-	4700 3250 4100 3250
-Wire Wire Line
-	4100 3250 4100 3700
-Connection ~ 4700 3250
 $Comp
 L Regulator_Linear:AMS1117-5.0 U?
@@
 U 1 1 5CDD7FDC
 P 1850 4750
-F 0 "U?" H 1850 5631 50  0000 C CNN
-F 1 "FT230XS" H 1850 5540 50  0000 C CNN
+F 0 "U?" H 2100 5450 50  0000 C CNN
+F 1 "FT230XS" H 2200 5350 50  0000 C CNN
 F 2 "Package_SO:SSOP-16_3.9x4.9mm_P0.635mm" H 2300 4100 50  0001 C CNN
 F 3 "http://www.ftdichip.com/Products/ICs/FT230X.html" H 1850 4750 50  0001 C CNN
 	1    1850 4750
-	1    0    0    -1
-$EndComp
-$Comp
-L Driver_Motor:DRV8848 U?
-U 1 1 5CDD91C7
-P 5400 1650
-F 0 "U?" H 5400 2431 50  0000 C CNN
-F 1 "DRV8848" H 5400 2340 50  0000 C CNN
-F 2 "Package_SO:TSSOP-16-1EP_4.4x5mm_P0.65mm" H 5400 950 50  0001 C CNN
-F 3 "http://www.ti.com/lit/ds/symlink/drv8848.pdf" H 4250 3000 50  0001 C CNN
-	1    5400 1650
 	1    0    0    -1
 $EndComp
@@
 L Device:Rotary_Encoder_Switch SW?
 U 1 1 5CDDCFA9
-P 8800 1550
-F 0 "SW?" H 8800 1917 50  0000 C CNN
-F 1 "Rotary_Encoder_Switch" H 8800 1826 50  0000 C CNN
-F 2 "" H 8650 1710 50  0001 C CNN
-F 3 "~" H 8800 1810 50  0001 C CNN
-	1    8800 1550
+P 6700 5300
+F 0 "SW?" H 6700 5667 50  0000 C CNN
+F 1 "Rotary_Encoder_Switch" H 6700 5576 50  0000 C CNN
+F 2 "" H 6550 5460 50  0001 C CNN
+F 3 "~" H 6700 5560 50  0001 C CNN
+	1    6700 5300
 	1    0    0    -1
 $EndComp
@@
 	0    -1   -1   0
 $EndComp
+Text GLabel 1300 950  1    50   Input ~ 0
+VDD
+Text GLabel 1900 1300 2    50   Input ~ 0
+GNDC
+Text GLabel 1100 1150 2    50   Input ~ 0
+GNDD
+Text GLabel 850  3000 2    50   Input ~ 0
+GNDC
+Text GLabel 700  3000 3    50   Input ~ 0
+GNDC
+Text GLabel 1100 2400 2    50   Input ~ 0
+VCC
+Text GLabel 4900 6250 2    50   Input ~ 0
+GNDC
+Text GLabel 1850 7050 2    50   Input ~ 0
+GNDC
 Wire Wire Line
-	6000 1850 6750 1850
+	1750 5450 1950 5450
 Wire Wire Line
-	6750 1850 6750 1800
-Wire Wire Line
-	6000 1950 6950 1950
-Wire Wire Line
-	6950 1950 6950 1800
-Wire Wire Line
-	6000 1450 6300 1450
-Wire Wire Line
-	6300 1450 6300 1600
-Wire Wire Line
-	6300 1600 6550 1600
-Wire Wire Line
-	6000 1550 6550 1550
-Wire Wire Line
-	6550 1550 6550 1400
+	1950 5450 2050 5450
+Connection ~ 1950 5450
+Text GLabel 2050 5450 2    50   Input ~ 0
+GNDC
+Text GLabel 1750 4050 1    50   Input ~ 0
+VCC
+Text GLabel 1950 4050 1    50   Input ~ 0
+VCC
+Text GLabel 4100 3700 0    50   Input ~ 0
+~RESET
+Text GLabel 1150 4950 0    50   Input ~ 0
+~RESET
+Text Notes 7000 7050 0    354  ~ 0
+Voight Focuser
+$Comp
+L JeffLibrary:DRV8825 U?
+U 1 1 5CDE1BDD
+P 4650 1550
+F 0 "U?" H 4675 2425 50  0000 C CNN
+F 1 "DRV8825" H 4675 2334 50  0000 C CNN
+F 2 "Package_SO:HTSSOP-28-1EP_4.4x9.7mm_P0.65mm_EP3.4x9.5mm_Mask2.4x6.17mm_ThermalVias" H 4750 650 50  0001 C CNN
+F 3 "http://www.ti.com/lit/ds/symlink/drv8825.pdf" H 4500 2200 50  0001 C CNN
+	1    4650 1550
+	1    0    0    -1
+$EndComp
+Wire Notes Line
+	8800 2050 8800 4050
+Wire Notes Line
+	8800 4050 10450 4050
+Wire Notes Line
+	10450 4050 10450 2050
+Wire Notes Line
+	10450 2050 8800 2050
 $EndSCHEMATC
