File: voightfocuser/_autosave-voightfocuser.sch (KiCad schematic (older format))
At the start: 28 parts

Commit message: new temperature
Parts:
- removed C?: .1uF, symbol Device:C
- removed U?: LM75B, symbol Sensor_Temperature:LM75B
- added U?: DHT11, Sensor:Aosong_DHT11_5.5x12.0_P2.54mm, symbol Sensor:DHT11
Changed lines of the file:
@@
 	2200 3850 2450 3850
-$Comp
-L Sensor_Temperature:LM75B U?
-U 1 1 5CDDA185
-P 9750 1450
-F 0 "U?" H 9550 1700 50  0000 C CNN
-F 1 "LM75B" H 9900 1700 50  0000 C CNN
-F 2 "" H 9750 1450 50  0001 C CNN
-F 3 "http://www.ti.com/lit/ds/symlink/lm75b.pdf" H 9750 1450 50  0001 C CNN
-	1    9750 1450
-	1    0    0    -1
-$EndComp
 $Comp
 L Device:Rotary_Encoder_Switch SW?
@@
 Text GLabel 1100 5250 2    50   Input ~ 0
 VCC5+
-Text GLabel 9750 1950 2    50   Input ~ 0
-GNDC
 $Comp
 L JeffLibrary:DRV8825 U?
@@
 Wire Wire Line
 	5050 1000 5250 1000
-Text GLabel 10050 900  2    50   Input ~ 0
-VCC5+
-Wire Wire Line
-	9750 950  9750 900
-Wire Wire Line
-	9750 900  10050 900
-Wire Notes Line
-	9000 650  10500 650
-Wire Notes Line
-	10500 650  10500 2050
-Wire Notes Line
-	9000 650  9000 2050
 Text Notes 9000 650  0    50   ~ 0
 Should be isolated from heat.\nBack of board on own ground plane.
@@
 	1    0    0    -1
 $EndComp
-Wire Notes Line
-	9000 2050 10500 2050
 $Comp
 L Interface_USB:FT230XS U?
@@
 	7100 5800 7150 5800
 $Comp
-L Device:C C?
-U 1 1 5CEAA16D
-P 9500 900
-F 0 "C?" V 9450 1000 50  0000 C CNN
-F 1 ".1uF" V 9550 1050 50  0000 C CNN
-F 2 "" H 9538 750 50  0001 C CNN
-F 3 "~" H 9500 900 50  0001 C CNN
-	1    9500 900
-	0    1    1    0
-$EndComp
-Text GLabel 9300 900  0    50   Input ~ 0
-GNDC
-Wire Wire Line
-	9300 900  9350 900
-Wire Wire Line
-	9650 900  9750 900
-Connection ~ 9750 900
+L Sensor:DHT11 U?
+U 1 1 5CEBE678
+P 9650 1450
+F 0 "U?" H 9406 1496 50  0000 R CNN
+F 1 "DHT11" H 9406 1405 50  0000 R CNN
+F 2 "Sensor:Aosong_DHT11_5.5x12.0_P2.54mm" H 9650 1050 50  0001 C CNN
+F 3 "http://akizukidenshi.com/download/ds/aosong/DHT11.pdf" H 9800 1700 50  0001 C CNN
+	1    9650 1450
+	1    0    0    -1
+$EndComp
 $EndSCHEMATC
