File: voightfocuser/voightfocuser.sch (KiCad schematic (older format))
At the start: 28 parts

Commit message: changed encoders. Added caps.
Parts:
- removed C?: .1uF, symbol Device:C
- removed U?: LM75B, symbol Sensor_Temperature:LM75B
- added C1, C3, C4: 47pF, Capacitor_SMD:C_0805_2012Metric_Pad1.15x1.40mm_HandSolder, symbol Device:C
- added C10, C16, C8: .1uF, Capacitor_SMD:C_0805_2012Metric_Pad1.15x1.40mm_HandSolder, symbol Device:C
- added C18, C19: 22pF, Capacitor_SMD:C_0805_2012Metric_Pad1.15x1.40mm_HandSolder, symbol Device:C
- added C20, C21, C5, C?: .01uF, Capacitor_SMD:C_0805_2012Metric_Pad1.15x1.40mm_HandSolder, symbol Device:C
- added FB1: Ferrite_Bead, Ferrite_THT:LairdTech_28C0236-0JW-10, symbol Device:Ferrite_Bead_Small
- added R1, R2: 27R, symbol Device:R
- added R10, R12, R13, R14, R15, R16, R17, R3, R7, R8, R9, R?: 10k, symbol Device:R
- added SW1: SW_Push, symbol Switch:SW_Push
- added U6: DHT11, Sensor:Aosong_DHT11_5.5x12.0_P2.54mm, symbol Sensor:DHT11
- added Y1: 16MHz, Crystal:Crystal_SMD_HC49-SD_HandSoldering, symbol Device:Crystal_Small
- C11, C12, C13, C14, C15, C17, C2, C6, C7, C9: renamed from C?; footprint (none) -> Capacitor_SMD:C_0805_2012Metric_Pad1.15x1.40mm_HandSolder
- J1: renamed from J?; footprint (none) -> Connector_USB:USB_Micro-B_Amphenol_10103594-0001LF_Horizontal
- J2: renamed from J?; footprint (none) -> Connector_BarrelJack:BarrelJack_CUI_PJ-063AH_Horizontal
- J3: renamed from J?; value AVR-ISP-6 -> Programming Header; footprint (none) -> Connector_PinHeader_2.54mm:PinHeader_1x06_P2.54mm_Vertical
- R11, R4, R5, R6: renamed from R?; footprint (none) -> Resistor_SMD:R_0805_2012Metric_Pad1.15x1.40mm_HandSolder
- RV1: renamed from RV?; footprint (none) -> Potentiometer_SMD:Potentiometer_Bourns_TC33X_Vertical
- SW2: renamed from SW?; footprint (none) -> Rotary_Encoder:RotaryEncoder_Alps_EC12E-Switch_Vertical_H20mm
- gave numbers to parts that had none: 7
Connections:
- net labels added: ADC6, ADC7, DIR, ENC_SW, GND, HIGH, INT0, INT1, LOW, MED, MODE0, MODE1, MODE2, RX, RXD, STEP, TEMP, TERMA, TERMB, TX, TXD, VCC, ~CTS, ~ENABLE, ~RTS, ~SS
- net labels removed: ~RST
- wire segments 111 -> 211
Other:
- moved on the sheet: C6, J3, SW2

Commit message: changed encoders. Added caps.
Parts:
- removed SW3: SW_Rotary12, symbol Switch:SW_Rotary12
- added R1, R13, R14: 10k, Resistor_SMD:R_0805_2012Metric_Pad1.15x1.40mm_HandSolder, symbol Device:R
- added SW1: Limit Switch, Connector_PinHeader_2.54mm:PinHeader_1x02_P2.54mm_Vertical, symbol Switch:SW_SPST
- added SW4: SP5T, Connector_PinHeader_2.54mm:PinHeader_1x06_P2.54mm_Vertical, symbol VoightFocuser:SP5T
- R10: renamed from R9; footprint (none) -> Resistor_SMD:R_0805_2012Metric_Pad1.15x1.40mm_HandSolder
- R11: renamed from R10; footprint (none) -> Resistor_SMD:R_0805_2012Metric_Pad1.15x1.40mm_HandSolder
- R15: renamed from R12; footprint (none) -> Resistor_SMD:R_0805_2012Metric_Pad1.15x1.40mm_HandSolder
- R16: renamed from R13; footprint (none) -> Resistor_SMD:R_0805_2012Metric_Pad1.15x1.40mm_HandSolder
- R17: renamed from R14; footprint (none) -> Resistor_SMD:R_0805_2012Metric_Pad1.15x1.40mm_HandSolder
- R18: renamed from R15; footprint (none) -> Resistor_SMD:R_0805_2012Metric_Pad1.15x1.40mm_HandSolder
- R19: renamed from R16; footprint (none) -> Resistor_SMD:R_0805_2012Metric_Pad1.15x1.40mm_HandSolder
- R2: renamed from R1; footprint (none) -> Resistor_SMD:R_0805_2012Metric_Pad1.15x1.40mm_HandSolder
- R20: renamed from R?; footprint (none) -> Resistor_SMD:R_0805_2012Metric_Pad1.15x1.40mm_HandSolder
- R21: renamed from R17; footprint (none) -> Resistor_SMD:R_0805_2012Metric_Pad1.15x1.40mm_HandSolder
- R3: renamed from R2; footprint (none) -> Resistor_SMD:R_0805_2012Metric_Pad1.15x1.40mm_HandSolder
- R4: renamed from R3; footprint (none) -> Resistor_SMD:R_0805_2012Metric_Pad1.15x1.40mm_HandSolder
- R8: renamed from R7; footprint (none) -> Resistor_SMD:R_0805_2012Metric_Pad1.15x1.40mm_HandSolder
- R9: renamed from R8; footprint (none) -> Resistor_SMD:R_0805_2012Metric_Pad1.15x1.40mm_HandSolder
- SW2: renamed from SW1; footprint (none) -> Connector_PinHeader_2.54mm:PinHeader_1x02_P2.54mm_Vertical
- gave numbers to parts that had none: 1
- renumbered C20 to C21, C21 to C22, R11 to R12, R4 to R5, R5 to R6, R6 to R7, SW2 to SW3
Connections:
- net labels added: ISENA, ISENB, LIMIT, MEDHIGH, MEDLOW
- net labels removed: ADC6, ~SS
- wire segments 211 -> 230
- no-connect marks 0 -> 8
Other:
- moved on the sheet: C18, C19, R20, Y1

Commit message: routing
Parts:
- removed C6: 1uF, Capacitor_SMD:C_0805_2012Metric_Pad1.15x1.40mm_HandSolder, symbol Device:CP
- removed R20: 10k, Resistor_SMD:R_0805_2012Metric_Pad1.15x1.40mm_HandSolder, symbol Device:R
- removed U1: AMS1117-5, Package_TO_SOT_SMD:SOT-223-3_TabPin2, symbol Regulator_Linear:AMS1117-5.0
- removed U5: ATmega328PB-AU, Package_QFP:TQFP-32_7x7mm_P0.8mm, symbol MCU_Microchip_ATmega:ATmega328PB-AU
- added SW2: SW_SPDT, Button_Switch_THT:SW_Slide_1P2T_CK_OS102011MS2Q, symbol Switch:SW_SPDT
- added U4: ATmega328P-AU, Package_QFP:TQFP-32_7x7mm_P0.8mm, symbol MCU_Microchip_ATmega:ATmega328P-AU
- C20: renamed from C21; value .01uF -> .1uF
- C21: renamed from C22; value .01uF -> .1uF
- Y1: footprint Crystal:Crystal_SMD_HC49-SD_HandSoldering -> Crystal:Crystal_SMD_HC49-SD
- renumbered C3 to C1, C14 to C10, C16 to C14, C17 to C16, C18 to C17, C19 to C18, C20 to C19, C4 to C2, C5 to C3, C1 to C4, C2 to C5, C8 to C6, C10 to C7, C7 to C8, J2 to J1, J1 to J2, R9 to R10, R10 to R11, R11 to R12, R21 to R20, R12 to R5, R5 to R6, R6 to R7, R7 to R8, R8 to R9, SW2 to SW1, SW1 to SW3, SW3 to SW4, SW4 to SW5, U2 to U1, U4 to U2, U6 to U5
Connections:
- net VCC5+ is gone; now on net VCC: C16.2, FB1.1, J3.2 (VCC)
- net DIR: now also U4.14 (PB2)
- net ENC_SW: now also U4.2 (PD4)
- net GND: now also SW5.6 (INPUT), U2.7 (GND), U4.21 (GND), U4.3 (GND), U4.5 (GND)
- net HIGH: now also U4.25 (PC2)
- net INT0: now also U4.32 (PD2)
- net INT1: now also U4.1 (PD3)
- net LIMIT: now also U4.28 (PC5)
- net LOW: now also U4.19 (ADC6)
- net MED: now also U4.23 (PC0)
- net MEDHIGH: now also U4.24 (PC1)
- net MEDLOW: now also U4.22 (ADC7)
- net MISO: now also U4.16 (PB4)
- net MODE0: now also U4.11 (PD7)
- net MODE1: now also U4.10 (PD6)
- net MODE2: now also U4.9 (PD5)
- net MOSI: now also U4.15 (PB3)
- net RX: now also U4.30 (PD0)
- net SCK: now also U4.17 (PB5)
- net STEP: now also U4.12 (PB0)
- net TEMP: now also U4.27 (PC4)
- net TX: now also U4.31 (PD1)
- net VCC: now also U4.18 (AVCC), U4.20 (AREF), U4.4 (VCC), U4.6 (VCC)
- net VDD12+: now also SW2.2 (B); no longer J1.1
- net ~ENABLE: now also U4.13 (PB1)
- net ~RESET: now also U4.29 (~RESET~/PC6)
- net at C17.2, Y1.1: now also U4.7 (XTAL1/PB6)
- net at C18.2, Y1.2: now also U4.8 (XTAL2/PB7)
- net ISENA: no longer names the net of R7.1, U3.6 (ISENA)
- net ISENB: no longer names the net of R8.1, U3.9 (ISENB)
- new net +12V: J1.1, SW2.1 (A)
- no-connect marks 8 -> 11
Other:
- moved on the sheet: C1, C10, C14, C16, C17, C18, C19, C2, C20, C21, C3, C4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

Commit message: more route
Parts:
- U3: symbol JeffLibrary:DRV8825 -> voightfocuser-rescue:DRV8825-JeffLibrary
Changed lines of the file:
@@
 GND
 $Comp
-L JeffLibrary:DRV8825 U3
+L voightfocuser-rescue:DRV8825-JeffLibrary U3
 U 1 1 5CDE1BDD
 P 4600 1650

Commit message: bigger board. routing prototype finished?
Parts:
- removed R1: 10k, Resistor_SMD:R_0805_2012Metric_Pad1.15x1.40mm_HandSolder, symbol Device:R
Connections:
- net GND: now also SW3.1 (A)
- net INT0: now also C21.1, R18.2; no longer C20.2, R16.2
- net INT1: now also C20.2, R16.2; no longer C21.1, R18.2
- net XTAL_N: now reaches C17.2, U4.7 (XTAL1/PB6), Y1.1
- net XTAL_P: now reaches C18.2, U4.8 (XTAL2/PB7), Y1.2
Changed lines of the file:
@@
 $EndComp
 Text GLabel 950  3500 0    50   Input ~ 0
-VCC
-$Comp
-L Device:R R1
-U 1 1 5D65848B
-P 1100 3500
-F 0 "R1" V 1000 3500 50  0000 C CNN
-F 1 "10k" V 1100 3500 50  0000 C CNN
-F 2 "Resistor_SMD:R_0805_2012Metric_Pad1.15x1.40mm_HandSolder" V 1030 3500 50  0001 C CNN
-F 3 "~" H 1100 3500 50  0001 C CNN
-	1    1100 3500
-	0    1    1    0
-$EndComp
+GND
 Text GLabel 1850 3500 2    50   Input ~ 0
 LIMIT
@@
 	1    0    0    -1
 $EndComp
-Wire Wire Line
-	5500 7750 5650 7750
-Wire Wire Line
-	5500 7600 5650 7600
-Text GLabel 5500 7750 0    50   Input ~ 0
+Text GLabel 5500 7600 0    50   Input ~ 0
 TERMB
 Text GLabel 5650 7750 2    50   Input ~ 0
@@
 Text GLabel 5650 7600 2    50   Input ~ 0
 INT0
-Text GLabel 5500 7600 0    50   Input ~ 0
+Text GLabel 5500 7750 0    50   Input ~ 0
 TERMA
 Wire Wire Line
@@
 Text Label 1150 2500 0    50   ~ 0
 +12V
+Wire Wire Line
+	950  3500 1250 3500
+Text GLabel 7900 4250 1    50   Input ~ 0
+XTAL_N
+Text GLabel 7900 4450 3    50   Input ~ 0
+XTAL_P
+Wire Wire Line
+	5500 7600 5650 7600
+Wire Wire Line
+	5500 7750 5650 7750
 $EndSCHEMATC
