File: voightfocuser/voightfocuser.kicad_pcb (KiCad board)
At the start: 2 copper layers, 60 parts, among them J1 USB_B_Micro, J2 Barrel_Jack, J3 Programming Header, M1 Stepper_Motor_bipolar, SW1 Limit Switch, SW2 SW_Push, SW3 Rotary_Encoder_Switch, SW4 SP5T, U1 AMS1117-5, U2 FT230XS, U3 DRV8825, U4 TXB0104D, U5 ATmega328PB-AU, U6 DHT11, Y1 16MHz

Commit message: routing
Parts:
- removed C22: .01uF, Capacitor_SMD:C_0805_2012Metric_Pad1.15x1.40mm_HandSolder
- removed R21: 10k, Resistor_SMD:R_0805_2012Metric_Pad1.15x1.40mm_HandSolder
- removed U6: DHT11, Sensor:Aosong_DHT11_5.5x12.0_P2.54mm
- added SW5: SP5T, Connector_PinHeader_2.54mm:PinHeader_1x06_P2.54mm_Vertical, F.Cu at (129.3, 123.2)
- C17: value .1uF -> 22pF
- C19: value 22pF -> .01uF
- C2: value 10uF -> 47pF
- C20, C21: value .01uF -> .1uF
- C3: value 47pF -> .01uF
- C5: value .01uF -> 10uF
- C6: value 1uF -> .1uF
- C7: value 100uF -> .1uF
- C8: value .1uF -> 100uF
- J1: value USB_B_Micro -> Barrel_Jack; footprint Connector_USB:USB_Micro-B_Amphenol_10103594-0001LF_Horizontal -> Connector_BarrelJack:BarrelJack_CUI_PJ-063AH_Horizontal
- J2: value Barrel_Jack -> USB_B_Micro; footprint Connector_BarrelJack:BarrelJack_CUI_PJ-063AH_Horizontal -> Connector_USB:USB_Micro-B_Amphenol_10103594-0001LF_Horizontal
- R5: value 1M -> 10k
- R6: value 250m -> 1M
- R8: value 10k -> 250m
- SW1: value Limit Switch -> SW_Push
- SW2: value SW_Push -> SW_SPDT; footprint Connector_PinHeader_2.54mm:PinHeader_1x02_P2.54mm_Vertical -> Button_Switch_THT:SW_Slide_1P2T_CK_OS102011MS2Q
- SW3: value Rotary_Encoder_Switch -> Limit Switch; footprint Rotary_Encoder:RotaryEncoder_Alps_EC12E-Switch_Vertical_H20mm -> Connector_PinHeader_2.54mm:PinHeader_1x02_P2.54mm_Vertical
- SW4: value SP5T -> Rotary_Encoder_Switch; footprint Connector_PinHeader_2.54mm:PinHeader_1x06_P2.54mm_Vertical -> Rotary_Encoder:RotaryEncoder_Alps_EC12E-Switch_Vertical_H20mm
- U1: value AMS1117-5 -> FT230XS; footprint Package_TO_SOT_SMD:SOT-223-3_TabPin2 -> Package_SO:SSOP-16_3.9x4.9mm_P0.635mm
- U2: value FT230XS -> TXB0104D; footprint Package_SO:SSOP-16_3.9x4.9mm_P0.635mm -> Package_SO:SOIC-14_3.9x8.7mm_P1.27mm
- U4: value TXB0104D -> ATmega328P-AU; footprint Package_SO:SOIC-14_3.9x8.7mm_P1.27mm -> Package_QFP:TQFP-32_7x7mm_P0.8mm
- U5: value ATmega328PB-AU -> DHT11; footprint Package_QFP:TQFP-32_7x7mm_P0.8mm -> Sensor:Aosong_DHT11_5.5x12.0_P2.54mm; moved to B.Cu
- Y1: footprint Crystal:Crystal_SMD_HC49-SD_HandSoldering -> Crystal:Crystal_SMD_HC49-SD; moved to B.Cu
- moved M1 124.8 mm to (174.0, 81.0), turned to 90 degrees
- moved C9 123.5 mm to (181.6, 84.6), turned to 180 degrees
- moved C11 121.3 mm to (181.9, 89.9), turned to 180 degrees
- moved R6 116.8 mm to (178.6, 85.6), turned to 90 degrees
- moved R7 116.3 mm to (177.8, 89.7), turned to 90 degrees
- moved RV1 114.9 mm to (180.8, 104.6), turned to 90 degrees
- moved SW2 114.4 mm to (161.0, 80.6)
- moved C12 113.9 mm to (176.0, 85.6), turned to 90 degrees
- moved U3 111.1 mm to (176.8, 97.0), turned to 270 degrees
- moved R14 109.0 mm to (177.8, 106.9), turned to 90 degrees
- moved C13 107.9 mm to (169.7, 88.9), turned to 90 degrees
- moved R13 106.2 mm to (175.5, 106.9), turned to 90 degrees
- moved C15 103.8 mm to (173.2, 106.9), turned to 90 degrees
- moved C8 101.6 mm to (171.6, 88.9), turned to 90 degrees
- moved J1 98.5 mm to (151.7, 87.5), turned to 180 degrees
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Connections:
- C1 pad 2: Net-(C1-Pad2) -> D-
- C10 pad 1: GND -> 3V3OUT
- C10 pad 2: 3V3OUT -> GND
- C14 pad 1: 3V3OUT -> GND
- C14 pad 2: GND -> VCC
- C17 pad 2: VCC5+ -> Net-(C17-Pad2)
- C19 pad 1: GND -> Net-(C19-Pad1)
- C19 pad 2: Net-(C19-Pad2) -> GND
- C2 pad 1: VDD12+ -> D+
- C20 pad 1: Net-(C20-Pad1) -> GND
- C20 pad 2: GND -> INT0
- C21 pad 1: GND -> INT1
- C21 pad 2: INT0 -> GND
- C3 pad 2: D- -> ~RESET
- C4 pad 1: D+ -> GND
- C4 pad 2: GND -> Net-(C4-Pad2)
- C5 pad 1: GND -> VDD12+
- C5 pad 2: ~RESET -> GND
- C6 pad 1: VCC5+ -> VCC
- C7 pad 1: VDD12+ -> GND
- C7 pad 2: GND -> 3V3OUT
- C8 pad 1: VCC -> VDD12+
- FB1 pad 1: VCC5+ -> VCC
- FB1 pad 2: Net-(C1-Pad2) -> Net-(C4-Pad2)
- J1 pad 1: Net-(C1-Pad2) -> /+12V
- J1 pad 2: D- -> GND
- J2 pad 1: VDD12+ -> Net-(C4-Pad2)
- J2 pad 2: GND -> D-
- J3 pad 2: VCC5+ -> VCC
- R10 pad 2: /~RTS -> /RXD
- R11 pad 2: /~CTS -> /~RTS
- R12 pad 1: Net-(R12-Pad1) -> 3V3OUT
- R12 pad 2: 3V3OUT -> /~CTS
- R17 pad 1: Net-(C20-Pad1) -> Net-(C19-Pad1)
- R20 pad 1: Net-(R20-Pad1) -> TEMP
- R5 pad 1: Net-(C12-Pad1) -> Net-(R5-Pad1)
- R5 pad 2: VDD12+ -> 3V3OUT
- R6 pad 1: /ISENA -> Net-(C12-Pad1)
- R6 pad 2: GND -> VDD12+
- R7 pad 1: /ISENB -> Net-(R7-Pad1)
- R8 pad 1: 3V3OUT -> Net-(R8-Pad1)
- R8 pad 2: /TXD -> GND
- R9 pad 2: /RXD -> /TXD
- SW1 pad 1: Net-(R1-Pad1) -> GND
- SW1 pad 2: LIMIT -> ~RESET
- SW2 pad 1: GND -> /+12V
- SW2 pad 2: ~RESET -> VDD12+
- U1 pad 1: GND -> /TXD
- U1 pad 2: VCC5+ -> /~RTS
- U1 pad 3: VDD12+ -> 3V3OUT
- U2 pad 1: /TXD -> 3V3OUT
- U2 pad 10: 3V3OUT -> (no net)
- U2 pad 11: ~RESET -> (no net)
- U2 pad 12: VCC -> RX
- U2 pad 13: GND -> TX
- U2 pad 14: (no net) -> VCC
- U2 pad 2: /~RTS -> /TXD
- U2 pad 3: 3V3OUT -> /RXD
- U2 pad 4: /RXD -> /~RTS
- U2 pad 5: GND -> /~CTS
- U2 pad 6: /~CTS -> (no net)
- U2 pad 7: (no net) -> GND
- U2 pad 8: Net-(R3-Pad1) -> Net-(R5-Pad1)
- U2 pad 9: Net-(R2-Pad1) -> (no net)
- U3 pad 28: (no net) -> GND
- U3 pad 6: /ISENA -> Net-(R7-Pad1)
- U3 pad 9: /ISENB -> Net-(R8-Pad1)
- U4 pad 1: 3V3OUT -> INT1
- U4 pad 10: (no net) -> MODE1
- U4 pad 11: (no net) -> MODE0
- U4 pad 12: RX -> STEP
- U4 pad 13: TX -> ~ENABLE
- U4 pad 14: VCC -> DIR
- U4 pad 2: /TXD -> ENC_SW
- U4 pad 3: /RXD -> GND
- U4 pad 4: /~RTS -> VCC
- U4 pad 5: /~CTS -> GND
- U4 pad 6: (no net) -> VCC
- U4 pad 7: (no net) -> Net-(C17-Pad2)
- U4 pad 8: Net-(R12-Pad1) -> Net-(C18-Pad2)
- U4 pad 9: (no net) -> MODE2
- U5 pad 1: INT1 -> VCC
- U5 pad 2: ENC_SW -> TEMP
- U5 pad 3: GND -> (no net)
- U5 pad 4: VCC -> GND
- Y1 pad 1: Net-(C18-Pad2) -> Net-(C17-Pad2)
- Y1 pad 2: Net-(C19-Pad2) -> Net-(C18-Pad2)
Routing:
- net VCC: track 0.00 -> 84.0 mm, vias 0 -> 2
- net ~RESET: track 0.00 -> 56.5 mm, vias 0 -> 3
- net VDD12+: track 0.00 -> 45.2 mm
- net TEMP: track 0.00 -> 41.9 mm, vias 0 -> 2
- net MODE1: track 0.00 -> 30.0 mm
- net MODE0: track 0.00 -> 29.9 mm
- net MODE2: track 0.00 -> 29.8 mm
- net STEP: track 0.00 -> 29.7 mm
- net ~ENABLE: track 0.00 -> 29.5 mm
- net /~RTS: track 0.00 -> 29.4 mm, vias 0 -> 2
- net DIR: track 0.00 -> 29.4 mm
- net /RXD: track 0.00 -> 28.8 mm, vias 0 -> 1
- net 3V3OUT: track 0.00 -> 28.7 mm
- net /TXD: track 0.00 -> 23.6 mm, vias 0 -> 2
- net Net-(RV1-Pad2): track 0.00 -> 22.8 mm, vias 0 -> 2
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- added copper zone on B.Cu, net GND
- added copper zone on F.Cu, net GND
Other:
- board outline added: 69.9 x 47.2 mm
- net class Stepper added: clearance 0.2, trace_width 0.4, via_dia 0.000686, via_drill 0.00033
- board text added: "1"
- board text added: "2"
- board text added: "3"
- board text added: "4"
- board text added: "5"
- board text added: "GND"
- board text added: "MISO"
- board text added: "MOSI"
- board text added: "ON/OFF"
- board text added: "SCK"
- board text added: "VCC"
- board text added: "~RST"

Commit message: more route
Routing:
- net GND: track 2.04 -> 50.6 mm, vias 31 -> 40
- net /~CTS: track 4.15 -> 42.9 mm, vias 0 -> 2
- net LIMIT: track 0.00 -> 35.7 mm, vias 0 -> 1
- net ~RESET: track 56.5 -> 75.4 mm, vias 3 -> 6
- net 3V3OUT: track 28.7 -> 47.0 mm, vias 0 -> 2
- net VCC: track 84.0 -> 99.4 mm
- net D+: track 6.67 -> 11.4 mm
- net D-: track 6.66 -> 10.9 mm

Commit message: bigger board. routing prototype finished?
Parts:
- removed R1: 10k, Resistor_SMD:R_0805_2012Metric_Pad1.15x1.40mm_HandSolder
- Y1: moved to F.Cu
- moved SW5 51.6 mm to (167.8, 88.8), turned to 270 degrees
- moved C10 35.0 mm to (131.2, 82.8)
- moved SW3 34.9 mm to (174.4, 66.2)
- moved R5 34.1 mm to (133.2, 85.0), turned to 180 degrees
- moved SW4 31.7 mm to (139.8, 122.4), turned to 180 degrees
- moved U2 31.7 mm to (137.5, 90.8)
- moved C14 30.7 mm to (143.1, 84.7)
- moved C4 29.7 mm to (126.6, 67.8)
- moved C16 22.5 mm to (163.1, 117.7)
- moved RV1 22.2 mm to (183.4, 82.5), turned to 0 degrees
- moved R15 21.9 mm to (145.5, 122.6), turned to 0 degrees
- moved R19 21.5 mm to (145.5, 114.7), turned to 180 degrees
- moved C1 21.1 mm to (119.6, 72.4)
- moved C2 21.1 mm to (115.6, 72.4)
- moved J2 21.1 mm to (117.8, 66.6)
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Connections:
- net Net-(C17-Pad2) renamed XTAL_N
- net Net-(C18-Pad2) renamed XTAL_P
- C20 pad 2: INT0 -> INT1
- C21 pad 1: INT1 -> INT0
- R16 pad 2: INT0 -> INT1
- R18 pad 2: INT1 -> INT0
- SW3 pad 1: Net-(R1-Pad1) -> GND
Routing:
- net VCC: track 99.4 -> 274.9 mm, vias 2 -> 0
- net ~RESET: track 75.4 -> 159.7 mm, vias 6 -> 1
- net TEMP: track 41.9 -> 74.6 mm, vias 2 -> 1
- net V3P3OUT: track 17.8 -> 46.4 mm
- net MOSI: track 10.3 -> 35.2 mm
- net TX: track 9.30 -> 33.6 mm
- net VDD12+: track 45.2 -> 68.4 mm
- net RX: track 10.7 -> 30.4 mm
- net HIGH: track 0.00 -> 17.0 mm
- net Net-(R2-Pad1): track 18.3 -> 34.6 mm
- net MISO: track 7.90 -> 23.3 mm, vias 2 -> 0
- net Net-(RV1-Pad2): track 22.8 -> 7.58 mm, vias 2 -> 0
- net MEDHIGH: track 0.00 -> 15.1 mm
- net LOW: track 0.00 -> 14.4 mm
- net MED: track 0.00 -> 14.4 mm
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Other:
- board size 69.9 x 47.2 mm -> 95.1 x 64.9 mm
- net class Default: via_dia 0.000686 -> 0.8; via_drill 0.00033 -> 0.6
- net class Power: via_dia 0.1 -> 1; via_drill 0.05 -> 0.8
- net class Stepper removed

Commit message: routing
Parts:
- moved R14 18.0 mm to (176.1, 99.6), turned to 270 degrees
- moved R13 14.1 mm to (179.1, 99.6), turned to 270 degrees
- moved R8 5.21 mm to (186.4, 73.4)
- moved R7 5.08 mm to (189.0, 73.5)
Routing:
- net 3V3OUT: track 48.2 -> 70.4 mm
- net Net-(R14-Pad2): track 9.36 -> 25.3 mm, vias 0 -> 2
- net V3P3OUT: track 46.4 -> 31.0 mm, vias 2 -> 0
- net GND: track 39.3 -> 26.5 mm, vias 12 -> 15
- net Net-(R13-Pad2): track 19.8 -> 10.2 mm, vias 2 -> 0
- net VCC: track 274.9 -> 281.0 mm
- net Net-(R8-Pad1): track 10.2 -> 15.5 mm
- net Net-(R7-Pad1): track 10.2 -> 15.4 mm
- net LIMIT: track 49.9 -> 54.0 mm
- net TEMP: track 74.6 -> 75.9 mm
- net /TXD: track 19.2 -> 19.9 mm
- net /RXD: track 40.7 -> 41.3 mm
- net /~RTS: track 23.4 -> 23.9 mm
- net TX: track 33.6 -> 34.1 mm
